File: baitap1.sch (KiCad schematic (older format))
At the start: 1 part

Commit message: thaydoi2
Parts:
- added P?: C64AC, symbol C64AC
- added U?: 74CBTLV3861, symbol 74CBTLV3861
Changed lines of the file:
@@
+	1    0    0    -1
+$EndComp
+$Comp
+L 74CBTLV3861 U?
+U 1 1 5922AC20
+P 6000 2750
+F 0 "U?" H 6100 3350 50  0000 L CNN
+F 1 "74CBTLV3861" H 6050 2050 50  0000 L CNN
+F 2 "" H 6000 2750 50  0000 C CNN
+F 3 "" H 6000 2750 50  0000 C CNN
+	1    6000 2750
+	1    0    0    -1
+$EndComp
+$Comp
+L C64AC P?
+U 1 1 5922AC6F
+P 3100 4150
+F 0 "P?" H 3100 7450 50  0000 C CNN
+F 1 "C64AC" V 3350 4150 50  0000 C CNN
+F 2 "" H 3100 4150 50  0000 C CNN
+F 3 "" H 3100 4150 50  0000 C CNN
+	1    3100 4150
 	1    0    0    -1
 $EndComp
